File: hardware_2/ascender_board.brd (EAGLE design)
At the start: 93.6 x 82.9 mm, 141 parts, among them IC1 LM2937, IC2 MC33932, J1 455-1750-1-ND, Q1 8MHz, Q2 BSS123, Q3 BSS123, Q4 BSS123, U1 STM32F722XX, U2 I2C EEPROM, U3 SPARKFUN-DIGITALIC_LSM303C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

Commit message: common
Parts:
- moved R41 8.47 mm to (89.3, 13.7), turned to 90 degrees
- moved C28 6.07 mm to (90.7, 19.1), turned to 0 degrees
- moved U4 4.89 mm to (96.4, 18.3)
- moved R42 3.41 mm to (91.7, 15.8)
- moved BOOT 1.85 mm to (89.7, 52.2)
- moved C1 1.85 mm to (63.4, 45.7)
- moved C12 1.85 mm to (13.7, 16.3)
- moved C15 1.85 mm to (59.6, 27.3)
- moved C16 1.85 mm to (51.6, 23.2)
- moved C18 1.85 mm to (58.7, 6.65)
- moved C19 1.85 mm to (36.9, 13.0)
- moved C2 1.85 mm to (63.5, 42.2)
- moved C20 1.85 mm to (36.9, 6.15)
- moved C21 1.85 mm to (60.5, 14.8)
- moved C23 1.85 mm to (30.8, 3.35)
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Routing:
- net GND: track 832.5 -> 843.6 mm, vias 100 -> 98
- net +3V3: track 659.3 -> 666.5 mm, vias 32 -> 34
- net ENC_RIGHT_SDA: track 66.7 -> 71.3 mm, vias 1 -> 3
- net N$20: track 7.54 -> 4.38 mm
- net ENC_LEFT_SDA: track 50.7 -> 53.0 mm
- net N$34: track 3.63 -> 5.89 mm
- net ENC_LEFT_SCL: track 56.3 -> 58.4 mm
- net ENC_RIGHT_SCL: track 74.2 -> 74.4 mm, vias 3 -> 1
Other:
- board size 93.6 x 82.9 mm -> 97.8 x 82.9 mm
